File: msnanopcb.brd (EAGLE design)
At the start: 160 x 100 mm, 17 parts, among them IC1 LD117AD2MTR, IC3 LM386N-1, X1 STEREOJACK

Commit message: Add files via upload
Parts:
- removed IC2: (no value), ic-package:SOCKET-16
- removed PAD2: WIREPADSMD1,27-254, wirepad:SMD1,27-2,54
- removed SV1: (no value), con-lstb:MA04-1
- removed SV2, SV3: (no value), con-lstb:MA04-2
- removed SV4: (no value), 00-con-lstb_edited:MA03-1
- added 3V3, 5V, 9VIN: WIREPADSMD1,27-254, wirepad:SMD1,27-2,54
- added C3: 1000uf, rcl:E3,5-8
- added C7: 0.1uf, rcl:E2-5
- added DAC: (no value), ic-package:SOCKET-16
- added L1: 10, rcl:0204/7
- added L2, L3: 12k, rcl:0204/7
- added MIC: (no value), 00-con-lstb_edited:MA03-1
- added NRF1, NRF2: (no value), con-lstb:MA04-2
- added OLED: (no value), con-lstb:MA04-1
- added R1: (no value), rcl:RTRIM3296P
- added S2: (no value), switch-dil:DS-05
- moved IC1 76.5 mm to (20.3, 52.1), flipped to the bottom, turned to 270 degrees
- moved GND 72.7 mm to (50.8, 53.3), flipped to the bottom
- moved C5 67.9 mm to (21.6, 62.2), flipped to the bottom, turned to 90 degrees
- moved C4 65.4 mm to (27.9, 62.2), flipped to the bottom, turned to 270 degrees
- moved C2 62.9 mm to (34.3, 62.2), flipped to the bottom, turned to 90 degrees
- moved U$2 61.8 mm to (41.9, 52.1), flipped to the bottom, turned to 90 degrees
- moved C1 60.3 mm to (40.6, 62.2), flipped to the bottom, turned to 90 degrees
- moved S1 55.2 mm to (16.8, 19.4), turned to 180 degrees
- moved U$1 54.6 mm to (31.8, 21.1), flipped to the bottom
- moved IC3 50.3 mm to (15.2, 41.1), flipped to the bottom
- moved X1 39.5 mm to (0.89, 18.8)
Connections:
- removed net AUDIO: SV4.1
- removed net N$19: SV1.1
- removed net N$2: GND.1
- removed net N$20: SV1.2
- removed net N$21: SV1.3
- removed net N$22: SV1.4
- removed net N$23: IC2.1
- removed net N$24: IC2.2
- removed net N$25: IC2.3
- removed net N$26: IC2.4
- removed net N$27: IC2.5
- removed net N$28: IC2.6
- removed net N$29: IC2.7
- removed net N$30: IC2.8
- removed net N$31: IC2.16
- removed net N$32: IC2.15
- removed net N$33: IC2.14
- removed net N$34: IC2.13
- removed net N$35: IC2.12
- removed net N$36: IC2.11
- removed net N$37: IC2.10
- removed net N$38: IC2.9
- removed net N$39: X1.1
- removed net N$40: X1.2
- removed net N$41: X1.5
- new net AUDIN: MIC.1, U$1.A0
- new net AUDOUT: C3.+, X1.2, X1.5
- new net BATLVL: L2.2, L3.1, S2.6
- new net CE: NRF1.3, NRF2.3
- new net DACOUT: DAC.14, DAC.15, DAC.16, R1.1
- new net DB0: DAC.1, U$1.TX
- new net DB1: DAC.2, U$1.RX
- new net DB2: DAC.3, U$1.D2
- new net DB3: DAC.4, U$1.D3
- new net DB4: DAC.5, U$1.D4
- new net DB5: DAC.6, U$1.D5
- new net DB6: DAC.7, U$1.D6
- new net DB7: DAC.8, U$1.D7
- new net N$4: C3.-, IC3.5, L1.1
- new net N$9: C7.+, L1.2
- new net NANO3V3: 3V3.1, U$1.3V3
- new net NANO5V: 5V.1, U$1.5V
- new net POTIN: IC3.3, R1.2
- new net S1: S2.2, S2.5, U$1.A7
- new net S2: S2.3, U$1.A6
- new net S3: S2.4, U$1.A3
- new net S4: S2.1, U$1.A2
- new net SCL: OLED.3, U$1.A5
- new net SDA: OLED.4, U$1.A4
- net 3V3: now also MIC.3, NRF1.2, NRF2.2; no longer SV2.2, SV3.2
- net 5V: now also DAC.11, OLED.1, U$1.VIN; no longer SV4.3
- net 9VIN: now also 9VIN.1, L3.2; no longer PAD2.1
- net CE1: now also U$1.D8; no longer SV2.3
- net CE2: now also U$1.A1; no longer SV3.3
- net CSN1: now also NRF2.4, U$1.D9; no longer SV2.4
- net CSN2: now also NRF1.4, U$1.D10; no longer SV3.4
- net GND: now also C7.-, DAC.10, DAC.12, DAC.13, DAC.9, GND.1, IC3.2, L2.1, MIC.2, NRF1.1, NRF2.1, OLED.2, R1.3, S2.10, S2.7, S2.8, S2.9, U$1.GND1, U$1.GND2, X1.1; no longer SV2.1, SV3.1, SV4.2
- net IRQ1: now also NRF2.8; no longer SV2.8
- net IRQ2: now also NRF1.8; no longer SV3.8
- net MISO: now also NRF1.7, NRF2.7, U$1.D12; no longer SV2.7, SV3.7
- net MOSI: now also NRF1.6, NRF2.6, U$1.D11; no longer SV2.6, SV3.6
- net SCK: now also NRF1.5, NRF2.5, U$1.D13; no longer SV2.5, SV3.5
Routing:
- net 3V3: track 0.00 -> 136.8 mm, vias 0 -> 1
- net SCK: track 0.00 -> 117.9 mm
- net 9VIN: track 0.00 -> 112.1 mm
- net MOSI: track 0.00 -> 105.7 mm
- net MISO: track 0.00 -> 95.9 mm, vias 0 -> 1
- net CSN2: track 0.00 -> 90.7 mm
- net 9V: track 0.00 -> 84.5 mm, vias 0 -> 1
- net DB0: track 0.00 -> 76.2 mm, vias 0 -> 1
- net CSN1: track 0.00 -> 72.7 mm
- net 5V: track 0.00 -> 72.2 mm
- net SCL: track 0.00 -> 61.3 mm, vias 0 -> 1
- net SDA: track 0.00 -> 55.8 mm, vias 0 -> 1
- net NANO3V3: track 0.00 -> 55.6 mm
- net DB2: track 0.00 -> 52.5 mm, vias 0 -> 1
- net DB1: track 0.00 -> 51.7 mm, vias 0 -> 1
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- added copper zone on layer 1, net GND
- added copper zone on layer 16, net GND
Other:
- board size 160 x 100 mm -> 61 x 80.9 mm
- board text added: "APHYRE 1.0"
