File: msnanopcb.sch (EAGLE design)
At the start: 17 parts, among them IC1 LD117AD2MTR, IC3 LM386N-1, X1 STEREOJACK

Commit message: Add files via upload
Parts:
- added 3V3, 5V: WIREPADSMD1,27-254, wirepad:WIREPADSMD1,27-254
- added C3: 1000uf, rcl:CPOL-EUE3.5-8
- added C7: 0.1uf, rcl:CPOL-EUE2-5
- added L1: 10, rcl:L-EU0204/7
- added L2, L3: 12k, rcl:L-EU0204/7
- added R1: (no value), rcl:R-TRIMM3296P
- added S2: (no value), switch-dil:DS05
- renumbered IC2 to DAC, PAD2 to 9VIN, SV1 to OLED, SV2 to NRF2, SV3 to NRF1, SV4 to MIC
Connections:
- removed net AUDIO: MIC.1
- removed net N$19: OLED.1
- removed net N$2: GND.P
- removed net N$20: OLED.2
- removed net N$21: OLED.3
- removed net N$22: OLED.4
- removed net N$23: DAC.1
- removed net N$24: DAC.2
- removed net N$25: DAC.3
- removed net N$26: DAC.4
- removed net N$27: DAC.5
- removed net N$28: DAC.6
- removed net N$29: DAC.7
- removed net N$30: DAC.8
- removed net N$31: DAC.16
- removed net N$32: DAC.15
- removed net N$33: DAC.14
- removed net N$34: DAC.13
- removed net N$35: DAC.12
- removed net N$36: DAC.11
- removed net N$37: DAC.10
- removed net N$38: DAC.9
- removed net N$39: X1.1
- removed net N$40: X1.2
- removed net N$41: X1.5
- new net AUDIN: MIC.1, U$1.A0
- new net AUDOUT: C3.+, X1.2, X1.5
- new net BATLVL: L2.2, L3.1, S2.6
- new net CE: NRF1.3, NRF2.3
- new net DACOUT: DAC.14, DAC.15, DAC.16, R1.A
- new net DB0: DAC.1, U$1.TX
- new net DB1: DAC.2, U$1.RX
- new net DB2: DAC.3, U$1.D2
- new net DB3: DAC.4, U$1.D3
- new net DB4: DAC.5, U$1.D4
- new net DB5: DAC.6, U$1.D5
- new net DB6: DAC.7, U$1.D6
- new net DB7: DAC.8, U$1.D7
- new net N$4: C3.-, IC3.OUT, L1.1
- new net N$9: C7.+, L1.2
- new net NANO3V3: 3V3.P, U$1.3V3
- new net NANO5V: 5V.P, U$1.5V
- new net POTIN: IC3.+IN, R1.S
- new net S1: S2.2, S2.5, U$1.A7
- new net S2: S2.3, U$1.A6
- new net S3: S2.4, U$1.A3
- new net S4: S2.1, U$1.A2
- new net SCL: OLED.3, U$1.A5
- new net SDA: OLED.4, U$1.A4
- net 3V3: now also MIC.3
- net 5V: now also DAC.11, OLED.1, U$1.VIN; no longer MIC.3
- net 9VIN: now also L3.2
- net CE1: now also U$1.D8; no longer NRF2.3
- net CE2: now also U$1.A1; no longer NRF1.3
- net CSN1: now also U$1.D9
- net CSN2: now also U$1.D10
- net GND: now also C7.-, DAC.10, DAC.12, DAC.13, DAC.9, GND.P, IC3.-IN, IC3.GND, L2.1, OLED.2, R1.E, S2.10, S2.7, S2.8, S2.9, U$1.GND1, U$1.GND2, X1.1
- net MISO: now also U$1.D12
- net MOSI: now also U$1.D11
- net SCK: now also U$1.D13
Other:
- note added: "EXTRA SWITCHES"
